File: BB_LED_Tube.kicad_pcb (KiCad board)
At the start: 2 copper layers, 30 x 57.6 mm, 46 parts, among them U1 ESP32-WROOM-32, U2 MAX485E, U3 TPS54202DDC, U4 AP2112K-3.3

Commit message: added reverse voltage protection & more mounting holes
Parts:
- added D1: D_Small, Diode_SMD:D_SMB, F.Cu at (61.2, 121.5)
- added H3: MountingHole, MountingHole:MountingHole_2.7mm_M2.5, F.Cu at (83.4, 142.5)
- added H4: MountingHole, MountingHole:MountingHole_2.7mm_M2.5, F.Cu at (59.8, 142.3)
- moved DMX_A1 9.20 mm to (58.6, 105.3)
- moved DMX_B1 9.20 mm to (58.6, 108.7)
- moved LED_Data1 9.20 mm to (58.6, 113.1)
- moved GND6 9.20 mm to (58.6, 101.9)
- moved U2 8.64 mm to (70.4, 103.3)
- moved R2 8.49 mm to (74.2, 104.7)
- moved R4 4.84 mm to (74.2, 108.3), turned to 0 degrees
- moved R3 3.39 mm to (70.4, 108.3), turned to 0 degrees
Connections:
- VCC2 pad 1: VCC -> /VIN
Routing:
- net +5V: track 51.9 -> 40.1 mm, vias 2 -> 0
- net DMX RX: track 7.12 -> 14.8 mm
- net /LED_Data: track 20.8 -> 13.9 mm, vias 0 -> 1
- net /DMX A: track 17.2 -> 22.0 mm, vias 0 -> 1
- net /DMX B: track 22.2 -> 19.6 mm, vias 2 -> 1
- net DMX EN: track 13.7 -> 15.7 mm
- net /Flash: track 10.6 -> 11.4 mm
- net DMX TX: track 12.4 -> 13.0 mm
- net VCC: vias 1 -> 10
- net GND: vias 36 -> 38
- added copper zone on F.Cu, net /VIN
- added copper zone on F.Cu, net VCC
Other:
- board size 30 x 57.6 mm -> 30 x 63.6 mm
- board text added: "LED Stripes"
- board text added: "VIN"
- board text removed: "POWER"

Commit message: small update
Routing:
- net +3V3: track 20.5 -> 19.9 mm
- net DMX RX: track 14.8 -> 14.3 mm
Other:
- outline, holes or cut-outs redrawn

Commit message: added voltage shifter and exchanged RS485 chip
Parts:
- removed U2: MAX485E, Package_SO:SOIC-8_3.9x4.9mm_P1.27mm
- added C12: 1uF, Capacitor_SMD:C_0603_1608Metric, F.Cu at (73.4, 104.9)
- added JP1: noVLS, Jumper:SolderJumper-2_P1.3mm_Open_RoundedPad1.0x1.5mm, F.Cu at (74.6, 101.3)
- added R10: 10k, Resistor_SMD:R_0603_1608Metric, F.Cu at (68.0, 102.7)
- added R8: 100R, Resistor_SMD:R_0603_1608Metric, F.Cu at (62.4, 110.9)
- added R9: 10k, Resistor_SMD:R_0603_1608Metric, F.Cu at (71.2, 102.7)
- added U5: SN74LVC1T45DCK, Package_TO_SOT_SMD:SOT-363_SC-70-6, F.Cu at (77.4, 101.3)
- added U6: THVD1400D, Package_TO_SOT_SMD:SOT-583-8, F.Cu at (71.2, 104.9)
- moved 3V1 8.54 mm to (84.8, 96.3)
- moved C7 4.20 mm to (81.8, 104.3), turned to 180 degrees
- moved 5V1 3.97 mm to (84.8, 104.3)
- moved DMX_A1 3.40 mm to (58.6, 108.7)
- moved DMX_B1 3.40 mm to (58.6, 105.3)
- moved R4 3.00 mm to (71.2, 108.3), turned to -90 degrees
- moved R3 1.40 mm to (69.0, 108.3), turned to 90 degrees
- moved C9 1.04 mm to (81.0, 98.5), turned to 0 degrees
- moved R2 1.02 mm to (75.2, 104.9), turned to -90 degrees
- moved U4 0.97 mm to (81.0, 101.3), turned to 90 degrees
Connections:
- LED_Data1 pad 1: /LED_Data -> /LED Out
- U1 pad 23: /LED_Data -> unconnected-(U1-IO15-Pad23)
- U1 pad 27: unconnected-(U1-IO16-Pad27) -> LED_Data
Routing:
- net Net-(JP1-A): track 0.00 -> 20.8 mm, vias 0 -> 2
- net LED_Data: track 0.00 -> 14.8 mm, vias 0 -> 1
- net /LED_Data: track 13.5 -> 0.00 mm, vias 1 -> 0
- net DMX TX: track 12.7 -> 19.9 mm
- net /LED Out: track 0.00 -> 4.25 mm
- net /DMX A: track 21.5 -> 24.7 mm, vias 1 -> 2
- net /DMX B: track 19.6 -> 17.4 mm, vias 1 -> 0
- net DMX EN: track 15.5 -> 17.5 mm
- net GND: track 2.32 -> 4.25 mm, vias 38 -> 46
- net DMX RX: track 14.3 -> 12.7 mm
- net +3V3: track 19.9 -> 20.9 mm
Other:
- board text added: "LED Strips"
- board text removed: "LED Stripes"
